File: hardware/radio-thing.kicad_sch (KiCad schematic)
At the start: 84 parts, among them J1 USB-C, J2 LiPo 1S, J3 ST7796 3.5in SPI, J4 RADAR HEAD, J5 DEBUG UART, Q1 AO3401A, Q2 2N7002, Q3 2N7002, SW1 PWR, SW2 RESET, SW3 BOOT, SW4 UP, SW5 DOWN, SW6 OK, SW7 BACK, SW8 MODE, U1 USBLC6-2SC6, U2 BQ24074RGT, U3 MAX17048G+T10, U4 TPS63001, U5 TPS61202, U6 ESP32-S3-WROOM-1U-N8R8, U7 ISM330DHCX, U8 LIS2MDL, U9 DWM3000

Commit message: Cut display controls to 3 buttons centred under the screen
UP / OK / DOWN on a 20 mm pitch directly below the display. Holds give the
missing actions: UP 1.5 s = cycle mode, OK 1.5 s = back, OK 3 s = sleep.
Debouncer reports hold time (new test). GPIO7/15 freed to test pads.

Co-Authored-By: Claude Opus 5.5 <noreply@anthropic.com>
Claude-Session: https://claude.ai/code/session_01Qyypna6NiNd8puVy66YruE
Parts:
- removed SW7: BACK, Button_Switch_THT:SW_PUSH-12mm, symbol Switch:SW_Push
- removed SW8: MODE, Button_Switch_THT:SW_PUSH-12mm, symbol Switch:SW_Push
- added TP1: IO7, TestPoint:TestPoint_Pad_D1.5mm, symbol Connector:TestPoint
- added TP2: IO15, TestPoint:TestPoint_Pad_D1.5mm, symbol Connector:TestPoint
- SW4: Note (none) -> short = up/zoom in, hold = cycle mode
- SW5: Note (none) -> short = down/zoom out
- SW6: Note Fitted on both builds; pod's only button; deep-sleep wake -> Fitted on both builds; pod's only button; deep-sleep wake. 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
Connections:
- net BTN_BACK renamed SPARE_IO7
- net SPARE_IO7: now also TP1.1
- net BTN_MODE renamed SPARE_IO15
- net SPARE_IO15: now also TP2.1
Other:
- moved on the sheet: SW5, SW6
Changed lines of the file:
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@@
 		)
 	)
-	(label "BTN_BACK"
+	(label "SPARE_IO7"
 		(at 210.82 68.58 180)
 		(fields_autoplaced yes)
@@
 		)
 	)
-	(label "BTN_MODE"
+	(label "SPARE_IO15"
 		(at 210.82 88.9 180)
 		(fields_autoplaced yes)
@@
 			)
 		)
+		(property "Note" "short = up/zoom in, hold = cycle mode"
+			(at 408.94 198.12 0)
+			(effects
+				(font
+					(size 1.27 1.27)
+				)
+				(hide yes)
+			)
+		)
 		(pin "1"
 		)
@@
 		(dnp no)
 		(fields_autoplaced yes)
-		(property "Reference" "SW5"
+		(property "Reference" "SW6"
 			(at 410.21 208.28 0.0)
 			(effects
@@
 			)
 		)
-		(property "Value" "DOWN"
+		(property "Value" "OK"
 			(at 408.94 212.344 0.0)
 			(effects
@@
 			)
 		)
-		(property "Variant" "DISP"
+		(property "Variant" "BOTH"
+			(at 408.94 210.82 0)
+			(effects
+				(font
+					(size 1.27 1.27)
+				)
+				(hide yes)
+			)
+		)
+		(property "Note" "Fitted on both builds; pod's only button; deep-sleep wake. Hold 1.5 s = back, 3 s = sleep"
 			(at 408.94 210.82 0)
 			(effects
@@
 			(project "radio-thing"
 				(path "/95b886be-7bb8-bf84-ce35-c7d9b1fe507a"
-					(reference "SW5")
+					(reference "SW6")
 					(unit 1)
 				)
@@
 		)
 	)
-	(label "BTN_DOWN"
+	(label "BTN_OK"
 		(at 403.86 210.82 180)
 		(fields_autoplaced yes)
@@
 		(dnp no)
 		(fields_autoplaced yes)
-		(property "Reference" "SW6"
+		(property "Reference" "SW5"
 			(at 410.21 220.98 0.0)
 			(effects
@@
 			)
 		)
-		(property "Value" "OK"
+		(property "Value" "DOWN"
 			(at 408.94 225.044 0.0)
 			(effects
@@
 			)
 		)
-		(property "Variant" "BOTH"
+		(property "Variant" "DISP"
 			(at 408.94 223.52 0)
 			(effects
@@
 			)
 		)
-		(property "Note" "Fitted on both builds; pod's only button; deep-sleep wake"
+		(property "Note" "short = down/zoom out"
 			(at 408.94 223.52 0)
 			(effects
@@
 			(project "radio-thing"
 				(path "/95b886be-7bb8-bf84-ce35-c7d9b1fe507a"
-					(reference "SW6")
+					(reference "SW5")
 					(unit 1)
 				)
@@
 		)
 	)
-	(label "BTN_OK"
+	(label "BTN_DOWN"
 		(at 403.86 223.52 180)
 		(fields_autoplaced yes)
@@
 	)
 	(symbol
-		(lib_id "Switch:SW_Push")
-		(at 408.94 236.22 0)
+		(lib_id "Connector:TestPoint")
+		(at 403.86 236.22 0)
 		(unit 1)
 		(exclude_from_sim no)
-		(in_bom yes)
+		(in_bom no)
 		(on_board yes)
 		(dnp no)
 		(fields_autoplaced yes)
-		(property "Reference" "SW7"
-			(at 410.21 233.68 0.0)
+		(property "Reference" "TP1"
+			(at 403.86 229.362 0.0)
 			(effects
 				(font
@@
 			)
 		)
-		(property "Value" "BACK"
-			(at 408.94 237.744 0.0)
+		(property "Value" "IO7"
+			(at 403.86 231.14 0.0)
 			(effects
 				(font
@@
 			)
 		)
-		(property "Footprint" "Button_Switch_THT:SW_PUSH-12mm"
-			(at 408.94 231.14 0.0)
+		(property "Footprint" "TestPoint:TestPoint_Pad_D1.5mm"
+			(at 408.94 236.22 0.0)
 			(effects
 				(font
@@
 		)
 		(property "Datasheet" "~"
-			(at 408.94 231.14 0.0)
+			(at 408.94 236.22 0.0)
 			(effects
 				(font
@@
 			)
 		)
-		(property "Description" "Push button switch, generic, two pins"
-			(at 408.94 236.22 0.0)
+		(property "Description" "test point"
+			(at 403.86 236.22 0.0)
 			(effects
 				(font
@@
 			)
 		)
-		(property "Variant" "DISP"
-			(at 408.94 236.22 0)
+		(property "Variant" "BOTH"
+			(at 403.86 236.22 0)
 			(effects
 				(font
@@
 			)
 		)
-		(pin "1"
+		(property "Note" "spare GPIO7"
+			(at 403.86 236.22 0)
+			(effects
+				(font
+					(size 1.27 1.27)
+				)
+				(hide yes)
+			)
 		)
-		(pin "2"
+		(pin "1"
 		)
 		(instances
 			(project "radio-thing"
 				(path "/95b886be-7bb8-bf84-ce35-c7d9b1fe507a"
-					(reference "SW7")
+					(reference "TP1")
 					(unit 1)
 				)
@@
 		)
 	)
-	(label "BTN_BACK"
-		(at 403.86 236.22 180)
+	(label "SPARE_IO7"
+		(at 403.86 236.22 270)
 		(fields_autoplaced yes)
 		(effects
@@
 		)
 	)
-	(label "GND"
-		(at 414.02 236.22 0)
-		(fields_autoplaced yes)
-		(effects
-			(font
-				(size 1.0 1.0)
-			)
-			(justify left bottom)
-		)
-	)
 	(symbol
-		(lib_id "Switch:SW_Push")
-		(at 408.94 248.92 0)
+		(lib_id "Connector:TestPoint")
+		(at 403.86 248.92 0)
 		(unit 1)
 		(exclude_from_sim no)
-		(in_bom yes)
+		(in_bom no)
 		(on_board yes)
 		(dnp no)
 		(fields_autoplaced yes)
-		(property "Reference" "SW8"
-			(at 410.21 246.38 0.0)
+		(property "Reference" "TP2"
+			(at 403.86 242.062 0.0)
 			(effects
 				(font
@@
 			)
 		)
-		(property "Value" "MODE"
-			(at 408.94 250.444 0.0)
+		(property "Value" "IO15"
+			(at 403.86 243.84 0.0)
 			(effects
 				(font
@@
 			)
 		)
-		(property "Footprint" "Button_Switch_THT:SW_PUSH-12mm"
-			(at 408.94 243.84 0.0)
+		(property "Footprint" "TestPoint:TestPoint_Pad_D1.5mm"
+			(at 408.94 248.92 0.0)
 			(effects
 				(font
@@
 		)
 		(property "Datasheet" "~"
-			(at 408.94 243.84 0.0)
+			(at 408.94 248.92 0.0)
 			(effects
 				(font
@@
 			)
 		)
-		(property "Description" "Push button switch, generic, two pins"
-			(at 408.94 248.92 0.0)
+		(property "Description" "test point"
+			(at 403.86 248.92 0.0)
 			(effects
 				(font
@@
 			)
 		)
-		(property "Variant" "DISP"
-			(at 408.94 248.92 0)
+		(property "Variant" "BOTH"
+			(at 403.86 248.92 0)
 			(effects
 				(font
@@
 			)
 		)
-		(pin "1"
+		(property "Note" "spare GPIO15"
+			(at 403.86 248.92 0)
+			(effects
+				(font
+					(size 1.27 1.27)
+				)
+				(hide yes)
+			)
 		)
-		(pin "2"
+		(pin "1"
 		)
 		(instances
 			(project "radio-thing"
 				(path "/95b886be-7bb8-bf84-ce35-c7d9b1fe507a"
-					(reference "SW8")
+					(reference "TP2")
 					(unit 1)
 				)
@@
 		)
 	)
-	(label "BTN_MODE"
-		(at 403.86 248.92 180)
+	(label "SPARE_IO15"
+		(at 403.86 248.92 270)
 		(fields_autoplaced yes)
 		(effects
@@
 		)
 	)
-	(label "GND"
-		(at 414.02 248.92 0)
-		(fields_autoplaced yes)
-		(effects
-			(font
-				(size 1.0 1.0)
-			)
-			(justify left bottom)
-		)
-	)

Commit message: Hardware check: datasheet-verified fixes to charger, regulators, sensors, display, buzzer
Checked every from-memory value against manufacturer datasheets and fixed:
- BQ24074 ITERM 15k -> 3.0k (was terminating at 50%), ILIM -> ~0.9 A
- TPS63001 inductor 1.5 -> 2.2 uH, VINA RC filter; TPS61202 COUT 22 uF
- LIS2MDL C1 220 nF + 10 uF; MAX17048 VDD 100 nF
- Display (MSP3525/ST7796): powered from switched VSYS, LED pin driven
  directly (it is a logic input), SD_CS pulled high
- Buzzer from 3V3 through 15 ohm with flyback across the coil
- DWM3000 IRQ pull-down; 100 ohm series on detachable head UARTs
- M3 holes on the button tab; In2 freed for power/signal routing

Co-Authored-By: Claude Opus 5.5 <noreply@anthropic.com>
Claude-Session: https://claude.ai/code/session_01Qyypna6NiNd8puVy66YruE
Parts:
- removed Q1: AO3401A, Package_TO_SOT_SMD:SOT-23, symbol Transistor_FET:AO3401A
- removed Q2: 2N7002, Package_TO_SOT_SMD:SOT-23, symbol Transistor_FET:2N7002
- removed R16: 100k, Resistor_SMD:R_0402_1005Metric, symbol Device:R
- added C25: 10u, Capacitor_SMD:C_0603_1608Metric, symbol Device:C
- added H5, H6: M3, MountingHole:MountingHole_3.2mm_M3, symbol Mechanical:MountingHole
- added R23: 15, Resistor_SMD:R_0402_1005Metric, symbol Device:R
- added R24, R26, R27, R28, R29: 100, Resistor_SMD:R_0402_1005Metric, symbol Device:R
- added R25: 100k, Resistor_SMD:R_0402_1005Metric, symbol Device:R
- BZ1: value Magnetic 3V 6mm -> 3V magnetic transducer ~3 kHz; Note (none) -> external-drive coil (~8.5 ohm), 2-4 V, <=150 mA mean: drive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
- C11: value 10u -> 22u; Note (none) -> DS min ~5*L uF = 11 uF before DC-bias derating
- C20: value 100n -> 220n; Note C1 set/reset cap (verify value) -> LIS2MDL C1 = 220 nF, low ESR, right at pins 5/6 (DS Table 2)
- C5: value 1u -> 100n; Note (none) -> MAX17048 VDD bypass 0.1 uF per datasheet
- C7: Note VINA decoupling -> VINA filter cap
- D1: Note flyback -> flyback across the coil
- J3: Note Common red 3.5in ST7796 SPI module pinout - check your modu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 -> lcdwiki MSP3525/MSP3526 (ST7796) pinout. VCC feeds the modu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
- L1: value 1.5uH 2A -> 2.2uH Isat>=2A low DCR; Note (none) -> TPS6300x DS Table 1 uses 2.2 uH (VLF4012-2R2)
- R14: Note touch controller unused - keep deselected -> keep the module's SD card deselected (it shares MISO)
- R15: value 100k -> 100; Note (none) -> LED pin is a logic input (onboard BSS138 + 10k pull-up): hi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
- R4: value 1.5k -> 1.78k; Note ILIM = 1550/R ~= 1.03 A input limit -> ILIM = 1610/R ~= 0.9 A input limit (USB-C default 900 mA). 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
- R5: Note safety timer (verify against datasheet) -> fast-charge timer ~6.2 h, pre-charge ~37 min (DS 9.3.5.6)
- R6: value 15k -> 3.0k; Note termination current (verify against datasheet) -> termination = 10% of ICHG for any RISET (0.03*R_ITERM/R_ISE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
Connections:
- net BL_G is gone; now on net LCD_BL_CTL: R15.1
- net +3V3: now also C25.1, R23.1; no longer J3.1 (Pin_1), R15.2
- net DC_IRQ: now also R25.1
- net GND: now also C25.2, R25.2
- net HEADA_RX: now also R27.1; no longer J4.7 (Pin_7)
- net HEADA_TX: now also R26.1; no longer J4.6 (Pin_6)
- net HEADB_RX: now also R29.1; no longer J4.9 (Pin_9)
- net HEADB_TX: now also R28.1; no longer J4.8 (Pin_8)
- net LCD_LED: now also R15.2
- net PWR_EN: now also J3.1 (Pin_1)
- net VSYS: now also R24.1; no longer BZ1.1 (+), C7.1, D1.1 (K), U4.8 (VINA)
- net LCD_SD_CS: now reaches J3.14 (Pin_14)
- net LCD_SD_CS: now also R14.1
- net TOUCH_CS: no longer names the net of J3.11 (Pin_11)
- net TOUCH_CS: no longer R14.1
- new net BB_VINA: C7.1, R24.2, U4.8 (VINA)
- new net BZ_P: BZ1.1 (+), D1.1 (K), R23.2
- new net HA_RX_C: J4.7 (Pin_7), R27.2
- new net HA_TX_C: J4.6 (Pin_6), R26.2
- new net HB_RX_C: J4.9 (Pin_9), R29.2
- new net HB_TX_C: J4.8 (Pin_8), R28.2
Other:
- moved on the sheet: BZ1, C10, C11, C12, C13, C14, C22, C23, C24, C7, C8, C9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

Commit message: Route rev A board and add manufacturing outputs
- Cluster placement: each converter's inductor and caps, the sensors'
  decoupling, USB-C parts, head-ID network and LEDs sit at their IC pins
- Two-pass Freerouting (route.sh) + GND pours: 938 segments, 108 vias,
  0 unconnected, 0 electrical DRC errors, 0 schematic-parity issues
- Button tab: routed slots + bridges instead of a V-score (a V-cut would
  sever the button traces)
- Fixed USB-C orientation-join pattern, 0.35 mm edge keep-outs, solid GND
  on IC thermal pads, 0.3 mm power traces, silkscreen tidy-up
- Optional DWM3000 footprint moved to rev B (antenna keep-out blocked routing)
- fab/: Gerber+drill zip, BOM and CPL per build variant, board-corner origin

Co-Authored-By: Claude Opus 5.5 <noreply@anthropic.com>
Claude-Session: https://claude.ai/code/session_01Qyypna6NiNd8puVy66YruE
Parts:
- removed C22: 10u, Capacitor_SMD:C_0805_2012Metric, symbol Device:C
- removed C23: 100n, Capacitor_SMD:C_0402_1005Metric, symbol Device:C
- removed R25: 100k, Resistor_SMD:R_0402_1005Metric, symbol Device:R
- removed U9: DWM3000, RF_Module:DWM1000, symbol RF_Module:DWM3000
Connections:
- no-connect marks 31 -> 22
Other:
- note removed: "Optional pod-to-pod UWB ranging [OPT]"
- moved on the sheet: BZ1, D1, D2, D3, D4, H1, H2, H3, H4, H5, H6, J3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
